Commit message: my changes

File: description/robot_core.xacro (robot description, xacro)
@@ -1,6 +1,8 @@
 <?xml version="1.0"?>
 <robot xmlns:xacro="http://www.ros.org/wiki/xacro">
-    <link
-    name="Chassis">
+  <link name="base_link">
+  </link>
+  <link
+      name="Chassis">
     <inertial>
       <origin
@@ -39,4 +41,9 @@
     </collision>
   </link>
+  <joint name="Chassis_Joint" type="fixed">
+    <parent link="base_link"/>
+    <child link="Chassis"/>
+    <origin xyz="-0.071091 0 0.098" rpy="0 0 0"/>
+  </joint>
   <gazebo reference="Chassis">
     <material>Gazebo/Grey</material>

Commit message: my changes

File: description/robot_core.xacro (robot description, xacro)
@@ -49,4 +49,10 @@
     <material>Gazebo/Grey</material>
   </gazebo>
+  <joint name="imu_joint" type="fixed">
+    <parent link="Chassis"/>
+    <child link="imu_link"/>
+    <origin xyz="0.3 0 0" rpy="0 0 0"/>
+  </joint>
+  <link name="imu_link"/>
   <link
     name="Left_Wheel">
